File: kicad/cap-module.kicad_sch (KiCad schematic)
At the start: 8 parts, among them J1 Capacitor Socket, U1 RaspberryPi_Pico, U2 AD7747, U3 Picoprobe

Commit message: Connect/label Picoprobe debug nets
Connections:
- net DBG_SWCLK: now also U3.4 (GPIO2)
- net DBG_SWDIO: now also U3.5 (GPIO3)
- net DBG_UART_RX: now also U3.7 (GPIO5)
- net DBG_UART_TX: now also U3.6 (GPIO4)
- net DBG_VCC: now also U3.39 (VSYS)
- net GND: now also U3.13 (GND), U3.18 (GND), U3.23 (GND), U3.28 (GND), U3.3 (GND), U3.38 (GND), U3.8 (GND)
- net at NS1.2 (Shield), NS2.2 (Shield): no longer U2.3 (SHLD)
- new net: NS1.2 (Shield), NS2.2 (Shield), U2.3 (SHLD)
Changed lines of the file:
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@@
+    (stroke (width 0) (type default))
+  )
+  (wire (pts (xy 247.65 113.03) (xy 247.65 114.3))
     (stroke (width 0) (type default))
   )
@@
     (stroke (width 0) (type default))
   )
+  (wire (pts (xy 209.55 59.69) (xy 224.79 59.69))
+    (stroke (width 0) (type default))
+  )
   (wire (pts (xy 45.72 102.87) (xy 45.72 142.24))
     (stroke (width 0) (type default))
   )
+  (wire (pts (xy 215.9 30.48) (xy 247.65 30.48))
+    (stroke (width 0) (type default))
+  )
+  (wire (pts (xy 209.55 57.15) (xy 224.79 57.15))
+    (stroke (width 0) (type default))
+  )
   (wire (pts (xy 158.75 50.8) (xy 158.75 59.69))
     (stroke (width 0) (type default))
@@
   )
   (wire (pts (xy 111.76 55.88) (xy 153.67 55.88))
+    (stroke (width 0) (type default))
+  )
+  (wire (pts (xy 209.55 62.23) (xy 224.79 62.23))
     (stroke (width 0) (type default))
   )
@@
     (stroke (width 0) (type default))
   )
+  (wire (pts (xy 209.55 64.77) (xy 224.79 64.77))
+    (stroke (width 0) (type default))
+  )
   (wire (pts (xy 91.44 142.24) (xy 127 142.24))
     (stroke (width 0) (type default))
@@
     (stroke (width 0) (type default))
   )
+  (wire (pts (xy 247.65 30.48) (xy 247.65 34.29))
+    (stroke (width 0) (type default))
+  )
   (wire (pts (xy 120.65 69.85) (xy 135.89 69.85))
     (stroke (width 0) (type default))
@@
     (effects (font (size 1.27 1.27)) (justify left bottom))
   )
+  (label "DBG_UART_TX" (at 209.55 62.23 0) (fields_autoplaced)
+    (effects (font (size 1.27 1.27)) (justify left bottom))
+  )
+  (label "DBG_VCC" (at 215.9 30.48 0) (fields_autoplaced)
+    (effects (font (size 1.27 1.27)) (justify left bottom))
+  )
   (label "DBG_SWCLK" (at 120.65 69.85 0) (fields_autoplaced)
     (effects (font (size 1.27 1.27)) (justify left bottom))
   )
+  (label "DBG_UART_RX" (at 209.55 64.77 0) (fields_autoplaced)
+    (effects (font (size 1.27 1.27)) (justify left bottom))
+  )
   (label "DBG_SWDIO" (at 120.65 72.39 0) (fields_autoplaced)
+    (effects (font (size 1.27 1.27)) (justify left bottom))
+  )
+  (label "DBG_SWDIO" (at 209.55 59.69 0) (fields_autoplaced)
+    (effects (font (size 1.27 1.27)) (justify left bottom))
+  )
+  (label "DBG_SWCLK" (at 209.55 57.15 0) (fields_autoplaced)
     (effects (font (size 1.27 1.27)) (justify left bottom))
   )
@@
         )
       )
+    )
+  )
+  (symbol (lib_id "power:GND") (at 247.65 114.3 0) (unit 1)
+    (in_bom yes) (on_board yes) (dnp no)
+    (property "Reference" "#PWR04" (at 247.65 120.65 0)
+      (effects (font (size 1.27 1.27)) hide)
+    )
+    (property "Value" "GND" (at 247.65 118.11 0)
+      (effects (font (size 1.27 1.27)))
+    )
+    (property "Footprint" "" (at 247.65 114.3 0)
+      (effects (font (size 1.27 1.27)) hide)
+    )
+    (property "Datasheet" "" (at 247.65 114.3 0)
+      (effects (font (size 1.27 1.27)) hide)
+    )
+    (pin "1")
+    (instances
+      (project "cap-module"
+        (path "/2da8fa58-ccef-42b1-8320-baeb3fec91e3"
+          (reference "#PWR04") (unit 1)
+        )
+      )
